File: stereo_modulation_fx_motherboard.sch (KiCad schematic (older format))
At the start: 96 parts, among them J1 dry_out_A, J10 Conn_01x04_Male, J11 Conn_01x04_Male, J12 Conn_01x04_Male, J13 Conn_01x05_Male, J2 CV_out_A, J3 wet_in_A, J4 rez_CV_out_A, J5 dry_out_B, J6 CV_out_B, J7 wet_in_B, J8 rez_CV_out_B, J9 +5_volts_in, SW1 sweep_mode, SW2 invert_B, SW3 DPDT_on_on_on, U1 Teensy3.2, U10 DG419LDY, U11 DG419LDY, U2 CD74HC4067M, U3 MCP4822, U4 MCP4822, U5 TL072, U6 MCP6002-xSN, U7 TL072, U8 MCP6002-xSN, U9 CC3-0512DF-E

Commit message: move schematic blocks around, add LEDs
Parts:
- removed J13: Conn_01x05_Male, Connector_PinHeader_2.54mm:PinHeader_1x05_P2.54mm_Vertical, symbol Connector:Conn_01x05_Male
- added D1, D2: NeoPixel_THT, LED_THT:LED_D5.0mm-4_RGB, symbol LED:NeoPixel_THT
- added J13: Conn_01x03_Male, Connector_PinHeader_2.54mm:PinHeader_1x03_P2.54mm_Vertical, symbol Connector:Conn_01x03_Male
Connections:
- net +3V3: now also D1.3 (VDD), D2.3 (VDD)
- net CV_out_B: now also C3.1, U4.8 (VA); no longer C1.1, U4.6 (VB)
- net GNDA: now also D1.2 (GND), D2.2 (GND), J13.1 (Pin_1)
- net LED_serial: now also D1.4 (DIN)
- net footswitch_A: now also J13.2 (Pin_2)
- net footswitch_B: now also J13.3 (Pin_3)
- net rez_CV_out_B: now also C1.1, U4.6 (VB); no longer C3.1, U4.8 (VA)
- new net: D1.1 (DOUT), D2.4 (DIN)
Other:
- note added: "12 bit SPI DACs"
- note added: "CV mux"
- note added: "LEDs"
- note added: "SPI output"
- note added: "Teensy uC"
- note added: "analog input"
- note added: "bias of 2.12V and 2.16V is ideal.\nextra resistor pads R19 and R20 \nare for trimming if needed.\nthis isn't really all that critical."
- note added: "digital output"
- note added: "footswitch connector"
- note added: "input pullup"
- note added: "plug-in board connectors"
- note added: "power supply"
- note removed: "12 bit DACs"
- note removed: "LED and footswitch connector"
- note removed: "between 2.12V and 2.16V is ideal.\nextra resistor pads R19 and R20 are for trimming if needed.\nthis isn't really all that critical."
- note removed: "demux"
- moved on the sheet: C1, C10, C11, C12, C13, C14, C15, C16, C17, C18, C19, C2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

Commit message: plug in boards are smaller now
Parts:
- removed J12: Conn_01x04_Male, Connector_PinHeader_2.54mm:PinHeader_1x04_P2.54mm_Vertical, symbol Connector:Conn_01x04_Male
- removed J13: Conn_01x03_Male, Connector_PinHeader_2.54mm:PinHeader_1x03_P2.54mm_Vertical, symbol Connector:Conn_01x03_Male
- added C40, C41, C42, C43, C44, C45, C7, C8, C9: 100nF, Capacitor_SMD:C_0805_2012Metric_Pad1.15x1.40mm_HandSolder, symbol Device:C
- added C5, C6: 4u7, Capacitor_SMD:C_0805_2012Metric_Pad1.15x1.40mm_HandSolder, symbol Device:CP1
- added J12, J14: Conn_01x03_Male, Connector_PinHeader_2.54mm:PinHeader_1x03_P2.54mm_Vertical, symbol Connector:Conn_01x03_Male
- added J13: Conn_01x04_Male, Connector_PinHeader_2.54mm:PinHeader_1x04_P2.54mm_Vertical, symbol Connector:Conn_01x04_Male
- added JP1: Jumper_NO_Small, Jumper:SolderJumper-2_P1.3mm_Open_RoundedPad1.0x1.5mm, symbol Device:Jumper_NO_Small
- added R21, R22: 2k2, Resistor_SMD:R_0805_2012Metric_Pad1.15x1.40mm_HandSolder, symbol Device:R
- added RV13, RV14: 100k, Potentiometer_SMD:Potentiometer_Bourns_3269W_Vertical, symbol Device:R_POT_TRIM
- added U12: MCP6002-xSN, Package_SO:SOIC-8_3.9x4.9mm_P1.27mm, symbol Amplifier_Operational:MCP6002-xSN
- C20, C21, C22, C23, C24, C25: footprint (none) -> Capacitor_SMD:C_0805_2012Metric_Pad1.15x1.40mm_HandSolder
- C33, C34, C35, C36: value C -> 100nF
- J9: footprint (none) -> Connector_PinHeader_2.54mm:PinHeader_1x02_P2.54mm_Vertical
- L1, L2, L3: footprint (none) -> Inductor_SMD:L_0805_2012Metric_Pad1.15x1.40mm_HandSolder
- R10, R9: value ??? -> 10k
- R11, R12: value 10k -> 30k
- R3, R4: value ??? -> 20k
- SW1: value sweep_mode -> sweep_mode_center_off
- SW3: value DPDT_on_on_on -> B_input_selector_on_on_on
Connections:
- net +12V: now also C32.1, R19.1, R20.1, C8.1
- net +3V3: now also C34.1, C35.1, C36.1, C40.1, C41.1, C42.1, C43.1, C44.1, C45.1, C7.1, U12.8 (V+); no longer R11.1, R19.1
- net -12V: now also C33.1, C9.1
- net CV_amp_bias: no longer R19.2, R20.1
- net GNDA: now also C20.2, C21.2, C33.2, C34.2, C35.2, C36.2, J9.2 (Pin_2), U8.3 (+), U8.5 (+), U9.2 (RC), U9.3 (Vin-), C40.2, C41.2, C42.2, C43.2, C44.2, C45.2, C5.2, C6.2, C7.2, C8.2, C9.2, J12.3 (Pin_3), J13.2 (Pin_2), J13.4 (Pin_4), J14.3 (Pin_3), JP1.2, R21.2, R22.2, U12.4 (V-); no longer R12.2, R20.2
- net LFO_rate_CV_in: now also J12.1 (Pin_1)
- net dry_A: now also R4.2, SW3.4; no longer C34.2, SW3.1
- net dry_B: now also R3.2; no longer C33.2
- net env_A: now also U2.20 (I11), RV14.1, U12.7; no longer C28.1, RV8.2, U2.6 (I3)
- net env_B: now also U2.21 (I10), RV13.1, U12.1; no longer C29.1, RV7.2, U2.3 (I6)
- net footswitch_A: now also J13.1 (Pin_1)
- net footswitch_B: now also J13.3 (Pin_3)
- net freq_CV_in: now also J14.1 (Pin_1)
- net wet_A: now also SW3.6; no longer SW3.4
- net at U11.2, U7.6 (-), U7.7: now also SW3.1; no longer SW3.6
- net Vin+: now reaches U1.33 (Vin)
- net Vin+: now also C20.1, J9.1 (Pin_1), L1.1
- net at U9.8 (case_1): now also JP1.1
- net at R3.1, R9.2, U8.2 (-): no longer C36.2
- net at R10.2, R4.1, U8.6 (-): no longer C35.2
- removed net A_to_uC: C36.1, R9.1, U2.20 (I11), U8.1
- removed net B_to_uC: C35.1, R10.1, U2.21 (I10), U8.7
- removed net audio_to_uC_amp_bias: C32.1, R11.2, R12.1, U8.3 (+), U8.5 (+)
- new net: J12.2 (Pin_2), R19.2
- new net: J14.2 (Pin_2), R20.2
- new net: C5.1, R11.1, R9.1, U12.3 (+)
- new net: R11.2, U8.1
- new net: R21.1, RV13.2, RV13.3, U12.2 (-)
- new net: R12.2, U8.7
- new net: C6.1, R10.1, R12.1, U12.5 (+)
- new net: R22.1, RV14.2, RV14.3, U12.6 (-)
- new net env_level_A: C28.1, RV8.2, U2.6 (I3)
- new net env_level_B: C29.1, RV7.2, U2.3 (I6)
- no-connect marks 0 -> 38
Other:
- note added: "LED indicators"
- note added: "R"
- note added: "R19 and R20 chosen to develop\n+5V accross a typical expression\npedal"
- note added: "S"
- note added: "T"
- note added: "TODO:\n\n-evaluate power supply\n\n-power input connector could be beefier\n\n-triple check all footprints!!!\n\n-evaluate MUX/DEMUX\n\n-add expression pedal stuff: resistor to V-, check biphase semi-clone for ideas"
- note added: "U8A and U8B are very simple\nfull wave rectifiers achieved by\nusing rail-to-rail opamps with \nspecific ratios of resistors"
- note added: "bias of 2.12V to\n2.16V is ideal.\n"
- note added: "center\ndetent"
- note added: "env A trim"
- note added: "env B trim"
- note added: "envelope followers"
- note added: "power supply and bypass caps"
- note removed: "LEDs"
- note removed: "TODO:\n\n-evaluate power supply\n\n-triple check all footprints!!!\n\n-figure out how to do the envelope follower/digitize the audio?\n\n- figure out CV in circuit\n\n-handle bypass switching (just do true bypass off-board?)\n\n-evaluate MUX/DEMUX\n\n-evaluate DACs (DACs work, but output max of 2.048 volts...\nthis might be fine, just need to scale it up on plug in boards...\nsee mcp4822_test in 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"
- note removed: "audio to uC amplifiers"
- note removed: "bias of 2.12V and 2.16V is ideal.\nextra resistor pads R19 and R20 \nare for trimming if needed.\nthis isn't really all that critical."
- note removed: "power supply"
- moved on the sheet: C1, C10, C11, C12, C13, C14, C15, C16, C17, C18, C19, C2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

Commit message: tidy schematic, add stitching vias
Parts:
- added C? (x2): C, Capacitor_SMD:C_0805_2012Metric_Pad1.15x1.40mm_HandSolder, symbol Device:C
Connections:
- net +12V: now also C?.1
- net -12V: now also C?.1
- net GNDA: now also C?.2, C?.2
- net CV_out_A renamed freq_CV_A
- net CV_out_B renamed freq_CV_B
- net rez_CV_out_A renamed rez_CV_A
- net rez_CV_out_B renamed rez_CV_B
Other:
- note added: "input/output buffers and bypass switches"
- note removed: "input/output buffers"
- moved on the sheet: C1, C10, C11, C12, C13, C14, C15, C16, C17, C18, C19, C2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
