File: kicad_docs/stereo_modulation_fx_motherboard.kicad_pcb (KiCad board)
At the start: 2 copper layers, 101.6 x 139.7 mm, 116 parts, among them J1 dry_out_A, J10 Conn_01x04_Male, J11 Conn_01x04_Male, J12 Conn_01x03_Male, J13 Conn_01x04_Male, J14 Conn_01x03_Male, J2 CV_out_A, J3 wet_in_A, J4 rez_CV_out_A, J5 dry_out_B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

Commit message: restrucure files, begin firmware
Parts:
- added C46: C, Capacitor_SMD:C_0805_2012Metric_Pad1.15x1.40mm_HandSolder, B.Cu at (54.4, 159.0)
- added C47: C, Capacitor_SMD:C_0805_2012Metric_Pad1.15x1.40mm_HandSolder, B.Cu at (57.1, 156.0)
- moved R20 32.6 mm to (112.8, 112.5)
- moved J14 26.7 mm to (124.5, 111.8), turned to 180 degrees
- moved J12 8.95 mm to (124.5, 84.1), turned to 180 degrees
- moved R19 5.06 mm to (112.8, 86.1)
- moved R14 0.76 mm to (105.9, 85.6)
Connections:
- net input_A renamed Net-(C26-Pad2)
- net input_B renamed Net-(C27-Pad2)
- net output_A renamed Net-(J11-Pad1)
- net output_B renamed Net-(J11-Pad3)
- net wet_B renamed Net-(J7-Pad3)
Routing:
- net +12V: track 289.4 -> 320.2 mm, vias 1 -> 3
- net freq_CV_in: track 20.8 -> 35.8 mm, vias 0 -> 1
- net LFO_rate_CV_in: track 10.2 -> 19.6 mm
- net Net-(J14-Pad2): track 2.91 -> 11.5 mm
- net Net-(J12-Pad2): track 3.81 -> 11.9 mm
- net Net-(C37-Pad2): track 15.0 -> 13.5 mm
- net wet_A: track 129.8 -> 131.2 mm
- net Vin-: vias 13 -> 201
