File: kicad_docs/stereo_modulation_fx_motherboard.sch (KiCad schematic (older format))
At the start: 118 parts, among them J1 dry_out_A, J10 Conn_01x04_Male, J11 Conn_01x04_Male, J12 rate_CV_in, J13 Conn_01x04_Male, J14 freq_CV_in, J2 CV_out_A, J3 wet_in_A, J4 rez_CV_out_A, J5 dry_out_B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

Commit message: begin BOM, add pdf of schematic
Parts:
- C30, C31: value 470nF -> 100nF
- C37, C38: value 4.7nF -> 10nF
- R1, R2: value 15k -> 100k
- R19, R20: value ??? -> selec
Other:
- note removed: "TODO:\n\n-evaluate power supply\n\n-power input connector could be beefier\n\n-triple check all footprints!!!\n\n-evaluate MUX/DEMUX\n\n-add expression pedal stuff: resistor to V-, check biphase semi-clone for ideas"
Changed lines of the file:
@@
 Sheet 1 1
 Title "stereo modulation FX motherboard"
-Date "2019-05-26"
+Date "2019-06-07"
 Rev "1"
 Comp ""
@@
 Wire Wire Line
 	6650 15150 7200 15150
-Text Notes 3900 -650 0    118  ~ 24
-TODO:\n\n-evaluate power supply\n\n-power input connector could be beefier\n\n-triple check all footprints!!!\n\n-evaluate MUX/DEMUX\n\n-add expression pedal stuff: resistor to V-, check biphase semi-clone for ideas
 $Comp
 L Amplifier_Operational:TL072 U7
@@
 P 19700 9500
 F 0 "R1" H 19770 9546 50  0000 L CNN
-F 1 "15k" V 19700 9450 50  0000 L CNN
+F 1 "100k" V 19700 9400 50  0000 L CNN
 F 2 "Resistor_SMD:R_0805_2012Metric_Pad1.15x1.40mm_HandSolder" V 19630 9500 50  0001 C CNN
 F 3 "~" H 19700 9500 50  0001 C CNN
@@
 P 19450 9250
 F 0 "C30" V 19350 9100 50  0000 C CNN
-F 1 "470nF" V 19350 9450 50  0000 C CNN
+F 1 "100nF" V 19350 9450 50  0000 C CNN
 F 2 "Capacitor_SMD:C_0805_2012Metric_Pad1.15x1.40mm_HandSolder" H 19488 9100 50  0001 C CNN
 F 3 "~" H 19450 9250 50  0001 C CNN
@@
 P 19700 11700
 F 0 "R2" H 19770 11746 50  0000 L CNN
-F 1 "15k" V 19700 11650 50  0000 L CNN
+F 1 "100k" V 19700 11600 50  0000 L CNN
 F 2 "Resistor_SMD:R_0805_2012Metric_Pad1.15x1.40mm_HandSolder" V 19630 11700 50  0001 C CNN
 F 3 "~" H 19700 11700 50  0001 C CNN
@@
 P 19450 11450
 F 0 "C31" V 19350 11300 50  0000 C CNN
-F 1 "470nF" V 19350 11650 50  0000 C CNN
+F 1 "100nF" V 19350 11650 50  0000 C CNN
 F 2 "Capacitor_SMD:C_0805_2012Metric_Pad1.15x1.40mm_HandSolder" H 19488 11300 50  0001 C CNN
 F 3 "~" H 19450 11450 50  0001 C CNN
@@
 P 3750 6750
 F 0 "C37" V 3650 6600 50  0000 C CNN
-F 1 "4.7nF" V 3650 6900 50  0000 C CNN
+F 1 "10nF" V 3650 6900 50  0000 C CNN
 F 2 "Capacitor_SMD:C_0805_2012Metric_Pad1.15x1.40mm_HandSolder" H 3788 6600 50  0001 C CNN
 F 3 "~" H 3750 6750 50  0001 C CNN
@@
 P 3800 7900
 F 0 "C38" V 3700 7750 50  0000 C CNN
-F 1 "4.7nF" V 3700 8050 50  0000 C CNN
+F 1 "10nF" V 3700 8050 50  0000 C CNN
 F 2 "Capacitor_SMD:C_0805_2012Metric_Pad1.15x1.40mm_HandSolder" H 3838 7750 50  0001 C CNN
 F 3 "~" H 3800 7900 50  0001 C CNN
@@
 P 2500 7050
 F 0 "R19" H 2650 7050 50  0000 C CNN
-F 1 "???" V 2500 7050 50  0000 C CNN
+F 1 "selec" V 2500 7050 50  0000 C CNN
 F 2 "Resistor_SMD:R_0805_2012Metric_Pad1.15x1.40mm_HandSolder" V 2430 7050 50  0001 C CNN
 F 3 "~" H 2500 7050 50  0001 C CNN
@@
 P 2500 8200
 F 0 "R20" H 2650 8200 50  0000 C CNN
-F 1 "???" V 2500 8200 50  0000 C CNN
+F 1 "selec" V 2500 8200 50  0000 C CNN
 F 2 "Resistor_SMD:R_0805_2012Metric_Pad1.15x1.40mm_HandSolder" V 2430 8200 50  0001 C CNN
 F 3 "~" H 2500 8200 50  0001 C CNN
